File: cercuit/Micropad.kicad_sch (KiCad schematic)
At the start: 28 parts, among them SW1 SW_Push, SW10 SW_Push, SW11 SW_Push, SW12 SW_Push, SW13 RotaryEncoder, SW14 RotaryEncoder, SW2 SW_Push, SW3 SW_Push, SW4 SW_Push, SW5 SW_Push, SW6 SW_Push, SW7 SW_Push, SW8 SW_Push, SW9 SW_Push

Commit message: updated the shchmatics swich placenmet and connected the pcb switch and diode
Parts:
- renumbered D4 to D10, D8 to D11, D5 to D2, D9 to D3, D2 to D4, D6 to D5, D10 to D6, D3 to D7, D7 to D8, D11 to D9, SW4 to SW10, SW8 to SW11, SW5 to SW2, SW9 to SW3, SW2 to SW4, SW6 to SW5, SW10 to SW6, SW3 to SW7, SW7 to SW8, SW11 to SW9
Changed lines of the file:
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@@
 		(dnp no)
 		(fields_autoplaced yes)
-		(property "Reference" "D8"
+		(property "Reference" "D11"
 			(at 64.77 106.6799 90)
 			(show_name no)
@@
 			(project "Micropad"
 				(path "/e75f1afd-22f0-4d62-bca3-34727f06bbde"
-					(reference "D8")
+					(reference "D11")
 					(unit 1)
 				)
@@
 		(dnp no)
 		(fields_autoplaced yes)
-		(property "Reference" "SW5"
+		(property "Reference" "SW2"
 			(at 57.15 58.42 0)
 			(show_name no)
@@
 			(project "Micropad"
 				(path "/e75f1afd-22f0-4d62-bca3-34727f06bbde"
-					(reference "SW5")
+					(reference "SW2")
 					(unit 1)
 				)
@@
 		(in_pos_files yes)
 		(dnp no)
-		(property "Reference" "D5"
+		(property "Reference" "D2"
 			(at 64.77 68.5799 90)
 			(show_name no)
@@
 			(project "Micropad"
 				(path "/e75f1afd-22f0-4d62-bca3-34727f06bbde"
-					(reference "D5")
+					(reference "D2")
 					(unit 1)
 				)
@@
 		(dnp no)
 		(fields_autoplaced yes)
-		(property "Reference" "SW11"
+		(property "Reference" "SW9"
 			(at 80.01 83.82 0)
 			(show_name no)
@@
 			(project "Micropad"
 				(path "/e75f1afd-22f0-4d62-bca3-34727f06bbde"
-					(reference "SW11")
+					(reference "SW9")
 					(unit 1)
 				)
@@
 		(dnp no)
 		(fields_autoplaced yes)
-		(property "Reference" "SW9"
+		(property "Reference" "SW3"
 			(at 80.01 58.42 0)
 			(show_name no)
@@
 			(project "Micropad"
 				(path "/e75f1afd-22f0-4d62-bca3-34727f06bbde"
-					(reference "SW9")
+					(reference "SW3")
 					(unit 1)
 				)
@@
 		(dnp no)
 		(fields_autoplaced yes)
-		(property "Reference" "SW4"
+		(property "Reference" "SW10"
 			(at 31.75 96.52 0)
 			(show_name no)
@@
 			(project "Micropad"
 				(path "/e75f1afd-22f0-4d62-bca3-34727f06bbde"
-					(reference "SW4")
+					(reference "SW10")
 					(unit 1)
 				)
@@
 		(in_pos_files yes)
 		(dnp no)
-		(property "Reference" "D9"
+		(property "Reference" "D3"
 			(at 87.63 68.5799 90)
 			(show_name no)
@@
 			(project "Micropad"
 				(path "/e75f1afd-22f0-4d62-bca3-34727f06bbde"
-					(reference "D9")
+					(reference "D3")
 					(unit 1)
 				)
@@
 		(dnp no)
 		(fields_autoplaced yes)
-		(property "Reference" "SW8"
+		(property "Reference" "SW11"
 			(at 57.15 96.52 0)
 			(show_name no)
@@
 			(project "Micropad"
 				(path "/e75f1afd-22f0-4d62-bca3-34727f06bbde"
-					(reference "SW8")
+					(reference "SW11")
 					(unit 1)
 				)
@@
 		(dnp no)
 		(fields_autoplaced yes)
-		(property "Reference" "D4"
+		(property "Reference" "D10"
 			(at 39.37 106.6799 90)
 			(show_name no)
@@
 			(project "Micropad"
 				(path "/e75f1afd-22f0-4d62-bca3-34727f06bbde"
-					(reference "D4")
+					(reference "D10")
 					(unit 1)
 				)
@@
 		(in_pos_files yes)
 		(dnp no)
-		(property "Reference" "D11"
+		(property "Reference" "D9"
 			(at 87.63 93.9799 90)
 			(show_name no)
@@
 			(project "Micropad"
 				(path "/e75f1afd-22f0-4d62-bca3-34727f06bbde"
-					(reference "D11")
+					(reference "D9")
 					(unit 1)
 				)
@@
 		(in_pos_files yes)
 		(dnp no)
-		(property "Reference" "D10"
+		(property "Reference" "D6"
 			(at 87.63 81.2799 90)
 			(show_name no)
@@
 			(project "Micropad"
 				(path "/e75f1afd-22f0-4d62-bca3-34727f06bbde"
-					(reference "D10")
+					(reference "D6")
 					(unit 1)
 				)
@@
 		(in_pos_files yes)
 		(dnp no)
-		(property "Reference" "D3"
+		(property "Reference" "D7"
 			(at 39.37 93.9799 90)
 			(show_name no)
@@
 			(project "Micropad"
 				(path "/e75f1afd-22f0-4d62-bca3-34727f06bbde"
-					(reference "D3")
+					(reference "D7")
 					(unit 1)
 				)
@@
 		(dnp no)
 		(fields_autoplaced yes)
-		(property "Reference" "SW10"
+		(property "Reference" "SW6"
 			(at 80.01 71.12 0)
 			(show_name no)
@@
 			(project "Micropad"
 				(path "/e75f1afd-22f0-4d62-bca3-34727f06bbde"
-					(reference "SW10")
+					(reference "SW6")
 					(unit 1)
 				)
@@
 		(dnp no)
 		(fields_autoplaced yes)
-		(property "Reference" "SW3"
+		(property "Reference" "SW7"
 			(at 31.75 83.82 0)
 			(show_name no)
@@
 			(project "Micropad"
 				(path "/e75f1afd-22f0-4d62-bca3-34727f06bbde"
-					(reference "SW3")
+					(reference "SW7")
 					(unit 1)
 				)
@@
 		(dnp no)
 		(fields_autoplaced yes)
-		(property "Reference" "SW7"
+		(property "Reference" "SW8"
 			(at 57.15 83.82 0)
 			(show_name no)
@@
 			(project "Micropad"
 				(path "/e75f1afd-22f0-4d62-bca3-34727f06bbde"
-					(reference "SW7")
+					(reference "SW8")
 					(unit 1)
 				)
@@
 		(in_pos_files yes)
 		(dnp no)
-		(property "Reference" "D6"
+		(property "Reference" "D5"
 			(at 64.77 81.2799 90)
 			(show_name no)
@@
 			(project "Micropad"
 				(path "/e75f1afd-22f0-4d62-bca3-34727f06bbde"
-					(reference "D6")
+					(reference "D5")
 					(unit 1)
 				)
@@
 		(dnp no)
 		(fields_autoplaced yes)
-		(property "Reference" "SW6"
+		(property "Reference" "SW5"
 			(at 57.15 71.12 0)
 			(show_name no)
@@
 			(project "Micropad"
 				(path "/e75f1afd-22f0-4d62-bca3-34727f06bbde"
-					(reference "SW6")
+					(reference "SW5")
 					(unit 1)
 				)
@@
 		(in_pos_files yes)
 		(dnp no)
-		(property "Reference" "D7"
+		(property "Reference" "D8"
 			(at 64.77 93.9799 90)
 			(show_name no)
@@
 			(project "Micropad"
 				(path "/e75f1afd-22f0-4d62-bca3-34727f06bbde"
-					(reference "D7")
+					(reference "D8")
 					(unit 1)
 				)
@@
 		(dnp no)
 		(fields_autoplaced yes)
-		(property "Reference" "SW2"
+		(property "Reference" "SW4"
 			(at 31.75 71.12 0)
 			(show_name no)
@@
 			(project "Micropad"
 				(path "/e75f1afd-22f0-4d62-bca3-34727f06bbde"
-					(reference "SW2")
+					(reference "SW4")
 					(unit 1)
 				)
@@
 		(in_pos_files yes)
 		(dnp no)
-		(property "Reference" "D2"
+		(property "Reference" "D4"
 			(at 39.37 81.2799 90)
 			(show_name no)
@@
 			(project "Micropad"
 				(path "/e75f1afd-22f0-4d62-bca3-34727f06bbde"
-					(reference "D2")
-					(unit 1)
-				)
+					(reference "D4")
+					(unit 1)
+				)

Commit message: key moddle
Parts:
- A1: footprint Module:RaspberryPi_Pico_Common_Unspecified -> Module:RaspberryPi_Pico_Common_THT
Changed lines of the file:
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@@
 			)
 		)
-		(property "Footprint" "Module:RaspberryPi_Pico_Common_Unspecified"
+		(property "Footprint" "Module:RaspberryPi_Pico_Common_THT"
 			(at 243.84 121.92 0)
 			(hide yes)
